File: driver-v0/driver-v0.kicad_pcb (KiCad board)
At the start: 2 copper layers, 45 x 40 mm, 16 parts, among them J1 Screw_Terminal_01x02, J2 Screw_Terminal_01x02, J3 Barrel_Jack, U1 DRV104PWP

Commit message: fix: change peak width from 150 us to 150 ms
max switching time is 100 ms
Parts:
- C4: value 18nF -> 0.18uF
Changed lines of the file:
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@@
     (tags "resistor")
     (property "Mfg" "Yageo")
-    (property "PartNum" "RC0805FR-0749K9L")
+    (property "PartNum" "RC0805FR-0749R9L")
     (property "Sheetfile" "driver-v0.kicad_sch")
     (property "Sheetname" "")
@@
     (tags "resistor")
     (property "Mfg" "Yageo")
-    (property "PartNum" "RC0805FR-0749K9L")
+    (property "PartNum" "RC0805JR-074K7L")
     (property "Sheetfile" "driver-v0.kicad_sch")
     (property "Sheetname" "")
@@
     (tags "capacitor")
     (property "Mfg" "KYOCERA AVX")
-    (property "PartNum" "KGM21NR71H183KT")
+    (property "PartNum" "08053C184KAT2A")
     (property "Sheetfile" "driver-v0.kicad_sch")
     (property "Sheetname" "")
@@
         (effects (font (size 1 1) (thickness 0.15)))
     )
-    (fp_text value "18nF" (at 0 1.68 90) (layer "F.Fab")
+    (fp_text value "0.18uF" (at 0 1.68 90) (layer "F.Fab")
         (effects (font (size 1 1) (thickness 0.15)))
     )
@@
     (descr "Barrel Jack, 2.0mm ID, 5.5mm OD, 24V, 8A, no switch, https://www.cui.com/product/resource/pj-063ah.pdf")
     (tags "barrel jack cui dc power")
-    (property "Mfg" "")
-    (property "PartNum" "")
-    (property "Sheetfile" "driver-v0.kicad_sch")
-    (property "Sheetname" "")
+    (property "Mfg" "CUI")
+    (property "PartNum" "PJ-063AH")
+    (property "Sheetfile" "driver-v0.kicad_sch")
+    (property "Sheetname" "")
