File: driver-v0/driver-v0.kicad_sch (KiCad schematic)
At the start: 16 parts, among them J1 Screw_Terminal_01x02, J2 Screw_Terminal_01x02, J3 Barrel_Jack, U1 DRV104PWP

Commit message: fix bom
Parts:
- R1: PartNum RC0805FR-0749K9L -> RC0805FR-0749R9L
- R5: PartNum RC0805FR-0749K9L -> RC0805JR-074K7L
Changed lines of the file:
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@@
       (effects (font (size 1.27 1.27)) hide)
     )
-    (property "PartNum" "RC0805FR-0749K9L" (at 81.28 105.664 0)
+    (property "PartNum" "RC0805FR-0749R9L" (at 81.28 105.664 0)
       (effects (font (size 1.27 1.27)) hide)
     )
@@
       (effects (font (size 1.27 1.27)) hide)
     )
-    (property "PartNum" "RC0805FR-0749K9L" (at 91.44 110.744 0)
-      (effects (font (size 1.27 1.27)) hide)
-    )
+    (property "PartNum" "RC0805JR-074K7L" (at 91.44 110.744 0)
+      (effects (font (size 1.27 1.27)) hide)
+    )

Commit message: fix: change peak width from 150 us to 150 ms
max switching time is 100 ms
Parts:
- C4: value 18nF -> 0.18uF; PartNum KGM21NR71H183KT -> 08053C184KAT2A
Other:
- note added: "150ms"
- note removed: "15us"
Changed lines of the file:
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@@
     (effects (font (size 1.27 1.27)) (justify left bottom))
   )
-  (text "15us" (at 113.03 98.552 0)
+  (text "150ms" (at 113.03 98.552 0)
     (effects (font (size 1.27 1.27)) (justify left bottom))
   )
@@
       (effects (font (size 1.27 1.27)))
     )
-    (property "Value" "18nF" (at 115.316 99.568 90)
+    (property "Value" "0.18uF" (at 116.586 99.568 90)
       (effects (font (size 1.27 1.27)))
     )
@@
       (effects (font (size 1.27 1.27)) hide)
     )
-    (property "PartNum" "KGM21NR71H183KT" (at 111.76 100.584 0)
+    (property "PartNum" "08053C184KAT2A" (at 111.76 100.584 0)
       (effects (font (size 1.27 1.27)) hide)
     )
